File: design/analog_front_end.sch (KiCad schematic (older format))
At the start: 17 parts, among them U1 ACS712

Commit message: Moving to PIVI 2.0, added circuits for current clamps
Parts:
- removed C22: 1nF, Capacitors_SMD:C_0603, symbol C
- removed C23: 100nF, Capacitors_SMD:C_0603, symbol C
- removed R16: 11.8k, Resistors_SMD:R_0603, symbol R
- removed R17: 3.16k, Resistors_SMD:R_0603, symbol R
- removed U1: ACS712, SOIC_Packages:SOIC-8_3.9x4.9mm_Pitch1.27mm, symbol ACS712
- R13: value 1k -> 10k
- R19: value 56k -> 10k
Connections:
- net labels removed: +5V, Current_AD, Phase_Out
- wire segments 31 -> 20
Other:
- note removed: "0.106 < Vdiv < 0.951\nViout = 0.106V when I = -20A\nViout = 0.528V when I = 0A\nViout = 0.951V when I = 20A"
- note removed: "0.5 < Viout < 4.5\nViout = 0.5V when I = -20A\nViout = 2.5V when I = 0A\nViout = 4.5V when I = 20A"
- note removed: "ACS712 datasheet in Application 4 recommends using a rectifier\ndiode when connecting Viout to an ADC. The only case where Viout can\nbe negative is when I is less than -20A. As we are protected by 20A\ncircuit breakers, Viout can never be negative so we can avoid the diodes,\nand just use a voltage divider."
- note removed: "ACS712ELCTR-20A-T"
- note removed: "Atmel App note uses a sunt R and two ADC input to measure current\nin both cycles. We don't want to use shunt resistors, instead we use Hall\nEffect current sensings ICs. We use only one AD channel per circuit.\nEach AD line can measure both cycles, as the sensor output offsets the\nvoltage to make it always positive.\n\nThis needs to be taken into account in the firmware."
- note removed: "Example resistors in DK:\n11.8k 1% 0.1W: 311-11.8KHRCT-ND\n3.16k 1% 0.1W: RHM3.16KCFCT-ND\n\n"
- note removed: "In ADC unsigned mode (single ended) Vmax = Vref * (1 - 0.05)\nWhen using Vref = 1V, Vmax = 0.95\nWe use 1V internal reference. It's a band gap reference,\nnot dependent on regulated power supply stability\n\nPlease note that AVR1631 uses differential signed mode for the current\nalso.\n\nSource: http://www.atmel.com/Images/Atmel-8032-Using-the-Atmel-AVR-XMEGA-ADC_Application-Note_AVR1300.pdf"
- note removed: "Vdiv"
- moved on the sheet: C1, C25, C26, L3, L9, R10, R11, R12, R13, R14, R15, R19
