File: design/ATXMEGA128A3U.sch (KiCad schematic (older format))
At the start: 20 parts, among them IC1 ATXMEGA128A3U-A, P1 CONN_02X05, X1 32.768kHz +/-20PPM 7pF SMD

Commit message: Moving to PIVI 2.0, added circuits for current clamps
Connections:
- wire segments 113 -> 117
Other:
- note added: "REVISAR ESTE SECTOR, RECONECTE LAS COSAS\n"

Commit message: Agrego los dos circuitos extra para medir tension
Other:
- note removed: "REVISAR ESTE SECTOR, RECONECTE LAS COSAS\n"
Changed lines of the file:
@@
 LIBS:memory
 LIBS:xilinx
-LIBS:special
 LIBS:microcontrollers
 LIBS:dsp
@@
 $Descr A4 11693 8268
 encoding utf-8
-Sheet 2 18
+Sheet 2 20
 Title "PIVI"
 Date "Mon 27 Jul 2015"
@@
 Wire Wire Line
 	8350 4150 8350 4050
-Wire Notes Line
-	9425 3125 9425 4825
-Wire Notes Line
-	9425 4825 8125 4825
-Wire Notes Line
-	8125 4825 8125 3125
-Wire Notes Line
-	8125 3125 9425 3125
-Text Notes 8125 4950 0    60   ~ 0
-REVISAR ESTE SECTOR, RECONECTE LAS COSAS\n
 Text HLabel 4920 2530 0    60   Input ~ 0
 RESET

Commit message: Edito conexiones pinza, agregado debub uart, agregado tension referencia
Parts:
- removed JP1: JUMPER, Pin_Headers:Pin_Header_Straight_1x02, symbol JUMPER
- renumbered L1 to L2, L17 to L3
Connections:
- no-connect marks 1 -> 2
