File: design/pivi-power-supply.sch (KiCad schematic (older format))
At the start: 3 parts, among them U7 TLV70233DBV

Commit message: Moving to PIVI 2.0, added circuits for current clamps
Changed lines of the file:
@@
 LIBS:txs0104e
 LIBS:less
+LIBS:pivi-shield-cache
 EELAYER 25 0
 EELAYER END
 $Descr A4 11693 8268
 encoding utf-8
-Sheet 8 12
+Sheet 10 18
 Title "PIVI"
-Date "sáb 01 nov 2014"
-Rev "1.0"
+Date "Mon 27 Jul 2015"
+Rev "2.0"
 Comp "Copyright (C) LESS industries S.A. 2014,2015"
 Comment1 "Share alike attribution non-commercial 4.0"
@@
 $EndComp
 Wire Wire Line
-	5650 3750 5650 3700
+	5650 3650 5650 3750
 Wire Wire Line
 	6850 3300 7150 3300
 Wire Wire Line
-	5650 3300 5650 3175
+	5650 3175 5650 3350
 Wire Wire Line
-	7150 3175 7150 3325
+	7150 3175 7150 3375
 $Comp
-L +5V #PWR057
+L +5V #PWR045
 U 1 1 548CBAAB
 P 5650 3175
-F 0 "#PWR057" H 5650 3265 20  0001 C CNN
+F 0 "#PWR045" H 5650 3265 20  0001 C CNN
 F 1 "+5V" H 5650 3300 30  0000 C CNN
 F 2 "" H 5650 3175 60  0000 C CNN
@@
 	6400 3750 6400 3650
 Wire Wire Line
-	7150 3775 7150 3725
+	7150 3675 7150 3775
 $Comp
-L +3V3 #PWR058
+L +3V3 #PWR046
 U 1 1 54965F4C
 P 7150 3175
-F 0 "#PWR058" H 7150 3025 60  0001 C CNN
+F 0 "#PWR046" H 7150 3025 60  0001 C CNN
 F 1 "+3V3" H 7150 3300 30  0000 C CNN
 F 2 "" H 7150 3175 60  0000 C CNN
@@
 $EndComp
 $Comp
-L GND #PWR059
+L GND #PWR047
 U 1 1 54BFA945
 P 5650 3750
-F 0 "#PWR059" H 5650 3500 60  0001 C CNN
+F 0 "#PWR047" H 5650 3500 60  0001 C CNN
 F 1 "GND" H 5650 3600 60  0000 C CNN
 F 2 "" H 5650 3750 60  0000 C CNN
@@
 $EndComp
 $Comp
-L GND #PWR060
+L GND #PWR048
 U 1 1 54BFA959
 P 6400 3750
-F 0 "#PWR060" H 6400 3500 60  0001 C CNN
+F 0 "#PWR048" H 6400 3500 60  0001 C CNN
 F 1 "GND" H 6400 3600 60  0000 C CNN
 F 2 "" H 6400 3750 60  0000 C CNN
@@
 $EndComp
 $Comp
-L GND #PWR061
+L GND #PWR049
 U 1 1 54BFA96D
 P 7150 3775
-F 0 "#PWR061" H 7150 3525 60  0001 C CNN
+F 0 "#PWR049" H 7150 3525 60  0001 C CNN
 F 1 "GND" H 7150 3625 60  0000 C CNN
 F 2 "" H 7150 3775 60  0000 C CNN
@@
 $EndComp
 Connection ~ 7150 3300
+Connection ~ 5650 3300
 $EndSCHEMATC

Commit message: Edito conexiones pinza, agregado debub uart, agregado tension referencia
Parts:
- renumbered C52 to C12, C53 to C13, U7 to U3
Changed lines of the file:
@@
 $EndDescr
 $Comp
-L TLV70233DBV U7
+L TLV70233DBV U3
 U 1 1 548CB80E
 P 6400 3350
-F 0 "U7" H 6150 3550 40  0000 C CNN
+F 0 "U3" H 6150 3550 40  0000 C CNN
 F 1 "TLV70233DBV" H 6500 3550 40  0000 C CNN
 F 2 "SMD_Packages:SOT-23-5" H 6400 3625 35  0000 C CIN
@@
 $EndComp
 $Comp
-L C C53
+L C C13
 U 1 1 548CB8AD
 P 7150 3525
-F 0 "C53" H 7175 3600 40  0000 L CNN
+F 0 "C13" H 7175 3600 40  0000 L CNN
 F 1 "1uF" H 7175 3425 40  0000 L CNN
 F 2 "Capacitors_SMD:C_0603" H 7450 3375 30  0000 C CNN
@@
 	7150 3175 7150 3375
 $Comp
-L +5V #PWR046
+L +5V #PWR44
 U 1 1 548CBAAB
 P 5650 3175
-F 0 "#PWR046" H 5650 3265 20  0001 C CNN
+F 0 "#PWR44" H 5650 3265 20  0001 C CNN
 F 1 "+5V" H 5650 3300 30  0000 C CNN
 F 2 "" H 5650 3175 60  0000 C CNN
@@
 $EndComp
 $Comp
-L C C52
+L C C12
 U 1 1 548CB868
 P 5650 3500
-F 0 "C52" H 5675 3575 40  0000 L CNN
+F 0 "C12" H 5675 3575 40  0000 L CNN
 F 1 "100nF" H 5675 3400 40  0000 L CNN
 F 2 "Capacitors_SMD:C_0603" H 5950 3325 30  0000 C CNN
@@
 	7150 3675 7150 3775
 $Comp
-L +3V3 #PWR047
+L +3V3 #PWR47
 U 1 1 54965F4C
 P 7150 3175
-F 0 "#PWR047" H 7150 3025 60  0001 C CNN
+F 0 "#PWR47" H 7150 3025 60  0001 C CNN
 F 1 "+3V3" H 7150 3300 30  0000 C CNN
 F 2 "" H 7150 3175 60  0000 C CNN
@@
 $EndComp
 $Comp
-L GND #PWR048
+L GND #PWR45
 U 1 1 54BFA945
 P 5650 3750
-F 0 "#PWR048" H 5650 3500 60  0001 C CNN
+F 0 "#PWR45" H 5650 3500 60  0001 C CNN
 F 1 "GND" H 5650 3600 60  0000 C CNN
 F 2 "" H 5650 3750 60  0000 C CNN
@@
 $EndComp
 $Comp
-L GND #PWR049
+L GND #PWR46
 U 1 1 54BFA959
 P 6400 3750
-F 0 "#PWR049" H 6400 3500 60  0001 C CNN
+F 0 "#PWR46" H 6400 3500 60  0001 C CNN
 F 1 "GND" H 6400 3600 60  0000 C CNN
 F 2 "" H 6400 3750 60  0000 C CNN
@@
 $EndComp
 $Comp
-L GND #PWR050
+L GND #PWR48
 U 1 1 54BFA96D
 P 7150 3775
-F 0 "#PWR050" H 7150 3525 60  0001 C CNN
+F 0 "#PWR48" H 7150 3525 60  0001 C CNN
 F 1 "GND" H 7150 3625 60  0000 C CNN
 F 2 "" H 7150 3775 60  0000 C CNN
